Commit message: Fix the bugs that kept 2D mapping from working
All of these were found by measuring against Gazebo ground truth rather than by
reading code, and each one alone is enough to stop a map from forming.

base_footprint sat 0.4 m below the floor, which made the map a 3.5 x 2.7 m patch
stuck to the robot. Three causes stacked:

  - quadruped_controller.cpp refused to publish foot contacts in simulation
    (`&& !in_gazebo_`). Without contacts the body-to-footprint EKF has nothing
    to stand on. The joint-states gate next to it is left alone - that one is
    correct, gz_ros2_control publishes those.
  - publish_foot_contacts was False in the launch file.
  - base_to_footprint.yaml fed the IMU's linear acceleration into the filter,
    so gravity was integrated into a steady downward drift. Roll and pitch only
    now, plus imu0_remove_gravitational_acceleration.

The scan then came out rotated ~100 degrees, which was a second-order effect of
the first fix: with every yaw input disabled the unobserved yaw state random
walks. pose0 keeps yaw true to anchor it. Leg odometry's yaw rate is disabled in
favour of the gyro's - the legs slip and cancel the IMU otherwise.

Also here:
  - robot_description is wrapped in ParameterValue(..., value_type=str) at all
    three sites, so launch stops trying to YAML-parse the URDF
  - /odom/ground_truth carries the Gazebo plugin's pose, bridged read-only and
    kept off the control path, so tests have something to measure against
  - the duplicate /cmd_vel bridge and the static map->odom and
    base_footprint->base_link publishers are removed - they competed with the
    EKF and with SLAM
  - sensor <visualize> flags off, gz_args gets -r so the world starts unpaused,
    and the default world is simple_room.sdf

Co-Authored-By: Claude Opus 5 <noreply@anthropic.com>

File: unitree_go2_description/urdf/unitree_go2_gazebo.xacro (robot description, xacro)
@@ -34,5 +34,7 @@
       <odom_frame>odom</odom_frame>
       <robot_base_frame>base_link</robot_base_frame>
-      <odom_topic>/odom</odom_topic>
+      <!-- Ground truth odometry. Deliberately not on /odom, which belongs to the
+           footprint_to_odom_ekf output. -->
+      <odom_topic>/odom/ground_truth</odom_topic>
       <odom_publish_frequency>50</odom_publish_frequency>
     </plugin>
@@ -43,5 +45,8 @@
       <always_on>true</always_on>
       <update_rate>100</update_rate>
-      <visualize>true</visualize>
+      <!-- Off by default: Gazebo draws sensor helper geometry over the robot,
+           which clutters the view and shows up in screenshots. RViz visualises
+           the same data properly. Set to true if you want it while debugging. -->
+      <visualize>false</visualize>
       <topic>imu/data</topic>
       <gz_frame_id>imu_link</gz_frame_id>
@@ -111,5 +116,5 @@
       <always_on>1</always_on>
       <update_rate>10</update_rate>
-      <visualize>1</visualize>
+      <visualize>0</visualize>
       <topic>rgb_image</topic>
     </sensor>

File: unitree_go2_description/urdf/unitree_go2_robot.xacro (robot description, xacro)
@@ -107,34 +107,4 @@
         <origin rpy="0 0 0" xyz="0.326 0 0.043"/>
     </joint>
-    <!-- <joint name="lidar_l1_joint" type="fixed">
-        <parent link="base_link"/>
-        <child link="lidar_l1_link"/>
-        <origin rpy="2.94 0 1.5705" xyz="0.25 -0.038 -0.03"/>
-    </joint>
-    <link name="lidar_l1_link">
-        <inertial>
-            <mass value="0.5"/>
-            <origin rpy="0 0 0" xyz="0 0 0"/>
-            <inertia ixx="0.01" ixy="0" ixz="0" iyy="0.01" iyz="0" izz="0.01"/>
-        </inertial>
-        <visual>
-            <origin rpy="0 0 0" xyz="0 0 0"/>
-            <geometry>
-                <mesh filename="file://$(find unitree_go2_description)/meshes/L1_4D_Lidar.dae" scale="1 1 1"/>
-            </geometry>
-            <material name="black">
-                <color rgba="0.0 0.0 0.0 1.0"/>
-            </material>
-        </visual>
-        <collision>
-            <origin rpy="0 0 0" xyz="0 0 0"/>
-            <geometry>
-                <mesh filename="file://$(find unitree_go2_description)/meshes/L1_4D_Lidar.dae" scale="1 1 1"/>
-            </geometry>
-            <material name="black">
-                <color rgba="0.0 0.0 0.0 1.0"/>
-            </material>
-        </collision>
-    </link> -->
     <xacro:leg name="rf" mirror="-1" mirror_dae= "False" front_hind="1" front_hind_dae="True" />
     <xacro:leg name="lf" mirror="1" mirror_dae="True" front_hind="1" front_hind_dae="True" />
